Commit message: feat: add TECHNICAL_REPORT.md, slam_explorer node, collision_monitor parameters, and launcher stability improvements

File: urdf/robot.urdf.xacro (robot description, xacro)
@@ -132,5 +132,5 @@
     <parent link="base_link"/>
     <child  link="caster_link"/>
-    <origin xyz="${-base_radius + caster_radius} 0 ${-base_height/2.0 + caster_radius}"
+    <origin xyz="${-base_radius + caster_radius} 0 ${-base_height/2.0 - wheel_radius + caster_radius}"
             rpy="0 0 0"/>
   </joint>
