Commit message: maping all rooms

File: install/delivery_robot/share/delivery_robot/urdf/robot.urdf.xacro (robot description, xacro)
@@ -1,273 +1 @@
-<?xml version="1.0"?>
-<!--
-  delivery_bot — Differential-Drive Mobile Robot
-  ================================================
-  A compact circular robot (radius 0.18 m) with:
-    • Two driven wheels (continuous joints) + one caster ball
-    • 360° 2D LIDAR at 10 Hz, 360 rays, 0.12–10 m range
-    • IMU sensor (for optional EKF fusion)
-    • Gazebo diff-drive plugin publishing /odom and /cmd_vel
-    • Full inertia tensors for realistic physics
--->
-<robot name="delivery_bot" xmlns:xacro="http://www.ros.org/wiki/xacro">
-  <!-- ═══════════════════════════════════════════════════════════════
-       PARAMETERS — change here, updates propagate everywhere
-  ═══════════════════════════════════════════════════════════════ -->
-  <xacro:property name="base_radius"    value="0.18"/>
-  <xacro:property name="base_height"    value="0.12"/>
-  <xacro:property name="base_mass"      value="5.0"/>
-  <xacro:property name="wheel_radius"   value="0.06"/>
-  <xacro:property name="wheel_width"    value="0.04"/>
-  <xacro:property name="wheel_mass"     value="0.5"/>
-  <xacro:property name="wheel_sep"      value="0.38"/>   <!-- track width -->
-  <xacro:property name="caster_radius"  value="0.025"/>
-  <xacro:property name="lidar_height"   value="0.11"/>   <!-- above base centre -->
-  <!-- Colours -->
-  <material name="dark_grey"><color rgba="0.2 0.2 0.2 1.0"/></material>
-  <material name="blue_body"><color rgba="0.1 0.4 0.8 1.0"/></material>
-  <material name="orange">   <color rgba="1.0 0.5 0.0 1.0"/></material>
-  <material name="black">    <color rgba="0.0 0.0 0.0 1.0"/></material>
-  <material name="red">      <color rgba="0.8 0.1 0.1 1.0"/></material>
-  <!-- ═══════════════════════════════════════════════════════════════
-       BASE FOOTPRINT  (virtual link — Nav2 convention)
-  ═══════════════════════════════════════════════════════════════ -->
-  <link name="base_footprint"/>
-  <joint name="base_footprint_joint" type="fixed">
-    <parent link="base_footprint"/>
-    <child  link="base_link"/>
-    <origin xyz="0 0 ${wheel_radius}" rpy="0 0 0"/>
-  </joint>
-  <!-- ═══════════════════════════════════════════════════════════════
-       BASE LINK  (robot chassis)
-  ═══════════════════════════════════════════════════════════════ -->
-  <link name="base_link">
-    <visual>
-      <geometry>
-        <cylinder radius="${base_radius}" length="${base_height}"/>
-      </geometry>
-      <material name="blue_body"/>
-    </visual>
-    <collision>
-      <geometry>
-        <cylinder radius="${base_radius}" length="${base_height}"/>
-      </geometry>
-    </collision>
-    <inertial>
-      <mass value="${base_mass}"/>
-      <!-- Solid cylinder: Ixx = Iyy = m(3r²+h²)/12 ; Izz = mr²/2 -->
-      <inertia
-        ixx="${base_mass*(3*base_radius*base_radius + base_height*base_height)/12.0}"
-        iyy="${base_mass*(3*base_radius*base_radius + base_height*base_height)/12.0}"
-        izz="${base_mass*base_radius*base_radius/2.0}"
-        ixy="0" ixz="0" iyz="0"/>
-    </inertial>
-  </link>
-  <!-- Gazebo colour for base -->
-  <gazebo reference="base_link">
-    <material>Gazebo/Blue</material>
-  </gazebo>
-  <!-- ═══════════════════════════════════════════════════════════════
-       WHEEL MACRO  — instantiated for left and right
-  ═══════════════════════════════════════════════════════════════ -->
-  <xacro:macro name="wheel" params="side y_reflect">
-    <link name="${side}_wheel">
-      <visual>
-        <origin rpy="${pi/2} 0 0" xyz="0 0 0"/>
-        <geometry>
-          <cylinder radius="${wheel_radius}" length="${wheel_width}"/>
-        </geometry>
-        <material name="dark_grey"/>
-      </visual>
-      <collision>
-        <origin rpy="${pi/2} 0 0" xyz="0 0 0"/>
-        <geometry>
-          <cylinder radius="${wheel_radius}" length="${wheel_width}"/>
-        </geometry>
-      </collision>
-      <inertial>
-        <mass value="${wheel_mass}"/>
-        <!-- Thin solid cylinder (wheel axis = Y): Ixx=Izz=m(3r²+h²)/12 ; Iyy=mr²/2 -->
-        <inertia
-          ixx="${wheel_mass*(3*wheel_radius*wheel_radius + wheel_width*wheel_width)/12.0}"
-          iyy="${wheel_mass*wheel_radius*wheel_radius/2.0}"
-          izz="${wheel_mass*(3*wheel_radius*wheel_radius + wheel_width*wheel_width)/12.0}"
-          ixy="0" ixz="0" iyz="0"/>
-      </inertial>
-    </link>
-    <joint name="${side}_wheel_joint" type="continuous">
-      <parent link="base_link"/>
-      <child  link="${side}_wheel"/>
-      <origin xyz="0 ${y_reflect * wheel_sep/2.0} ${-base_height/2.0 + wheel_radius - wheel_radius}"
-              rpy="0 0 0"/>
-      <axis xyz="0 1 0"/>
-      <dynamics damping="0.1" friction="0.05"/>
-    </joint>
-    <gazebo reference="${side}_wheel">
-      <material>Gazebo/DarkGrey</material>
-      <mu1>1.0</mu1>
-      <mu2>1.0</mu2>
-      <kp>500000.0</kp>
-      <kd>10.0</kd>
-    </gazebo>
-  </xacro:macro>
-  <xacro:wheel side="left"  y_reflect=" 1"/>
-  <xacro:wheel side="right" y_reflect="-1"/>
-  <!-- ═══════════════════════════════════════════════════════════════
-       CASTER WHEEL  (passive ball at rear)
-  ═══════════════════════════════════════════════════════════════ -->
-  <link name="caster_link">
-    <visual>
-      <geometry><sphere radius="${caster_radius}"/></geometry>
-      <material name="black"/>
-    </visual>
-    <collision>
-      <geometry><sphere radius="${caster_radius}"/></geometry>
-    </collision>
-    <inertial>
-      <mass value="0.1"/>
-      <inertia ixx="1e-5" iyy="1e-5" izz="1e-5" ixy="0" ixz="0" iyz="0"/>
-    </inertial>
-  </link>
-  <joint name="caster_joint" type="fixed">
-    <parent link="base_link"/>
-    <child  link="caster_link"/>
-    <origin xyz="${-base_radius + caster_radius} 0 ${-base_height/2.0 - wheel_radius + caster_radius}"
-            rpy="0 0 0"/>
-  </joint>
-  <gazebo reference="caster_link">
-    <material>Gazebo/Black</material>
-    <mu1>0.0</mu1>
-    <mu2>0.0</mu2>
-  </gazebo>
-  <!-- ═══════════════════════════════════════════════════════════════
-       LIDAR LINK
-  ═══════════════════════════════════════════════════════════════ -->
-  <link name="laser_link">
-    <visual>
-      <geometry>
-        <cylinder radius="0.04" length="0.04"/>
-      </geometry>
-      <material name="orange"/>
-    </visual>
-    <collision>
-      <geometry>
-        <cylinder radius="0.04" length="0.04"/>
-      </geometry>
-    </collision>
-    <inertial>
-      <mass value="0.1"/>
-      <inertia ixx="1e-5" iyy="1e-5" izz="1e-5" ixy="0" ixz="0" iyz="0"/>
-    </inertial>
-  </link>
-  <joint name="laser_joint" type="fixed">
-    <parent link="base_link"/>
-    <child  link="laser_link"/>
-    <origin xyz="0 0 ${base_height/2.0 + 0.02}" rpy="0 0 0"/>
-  </joint>
-  <gazebo reference="laser_link">
-    <material>Gazebo/Orange</material>
-    <!-- ── 360° LIDAR sensor plugin ── -->
-    <sensor type="ray" name="lidar_sensor">
-      <pose>0 0 0 0 0 0</pose>
-      <always_on>true</always_on>
-      <visualize>false</visualize>
-      <update_rate>10</update_rate>
-      <ray>
-        <scan>
-          <horizontal>
-            <samples>360</samples>
-            <resolution>1</resolution>
-            <min_angle>-3.14159265</min_angle>
-            <max_angle> 3.14159265</max_angle>
-          </horizontal>
-        </scan>
-        <range>
-          <min>0.12</min>
-          <max>10.0</max>
-          <resolution>0.01</resolution>
-        </range>
-        <noise>
-          <type>gaussian</type>
-          <mean>0.0</mean>
-          <stddev>0.01</stddev>
-        </noise>
-      </ray>
-      <plugin name="gazebo_ros_lidar" filename="libgazebo_ros_ray_sensor.so">
-        <ros>
-          <remapping>~/out:=/scan</remapping>
-        </ros>
-        <output_type>sensor_msgs/LaserScan</output_type>
-        <frame_name>laser_link</frame_name>
-      </plugin>
-    </sensor>
-  </gazebo>
-  <!-- ═══════════════════════════════════════════════════════════════
-       IMU LINK  (used by robot_localization EKF — optional)
-  ═══════════════════════════════════════════════════════════════ -->
-  <link name="imu_link">
-    <visual>
-      <geometry><box size="0.02 0.02 0.02"/></geometry>
-      <material name="red"/>
-    </visual>
-    <inertial>
-      <mass value="0.01"/>
-      <inertia ixx="1e-7" iyy="1e-7" izz="1e-7" ixy="0" ixz="0" iyz="0"/>
-    </inertial>
-  </link>
-  <joint name="imu_joint" type="fixed">
-    <parent link="base_link"/>
-    <child  link="imu_link"/>
-    <origin xyz="0 0 0" rpy="0 0 0"/>
-  </joint>
-  <gazebo reference="imu_link">
-    <sensor name="imu_sensor" type="imu">
-      <always_on>true</always_on>
-      <update_rate>100</update_rate>
-      <plugin name="gazebo_ros_imu" filename="libgazebo_ros_imu_sensor.so">
-        <ros>
-          <remapping>~/out:=/imu</remapping>
-        </ros>
-        <frame_name>imu_link</frame_name>
-      </plugin>
-    </sensor>
-  </gazebo>
-  <!-- ═══════════════════════════════════════════════════════════════
-       DIFFERENTIAL DRIVE PLUGIN
-       Subscribes: /cmd_vel  (geometry_msgs/Twist)
-       Publishes:  /odom     (nav_msgs/Odometry)
-                  /tf odom → base_footprint
-  ═══════════════════════════════════════════════════════════════ -->
-  <gazebo>
-    <plugin name="differential_drive_controller"
-            filename="libgazebo_ros_diff_drive.so">
-      <!-- Joints -->
-      <left_joint>left_wheel_joint</left_joint>
-      <right_joint>right_wheel_joint</right_joint>
-      <!-- Geometry -->
-      <wheel_separation>${wheel_sep}</wheel_separation>
-      <wheel_diameter>${2 * wheel_radius}</wheel_diameter>
-      <!-- Limits -->
-      <max_wheel_torque>20</max_wheel_torque>
-      <max_wheel_acceleration>1.0</max_wheel_acceleration>
-      <!-- Odometry -->
-      <publish_odom>true</publish_odom>
-      <publish_odom_tf>true</publish_odom_tf>
-      <publish_wheel_tf>false</publish_wheel_tf>
-      <!-- Frames -->
-      <odometry_frame>odom</odometry_frame>
-      <robot_base_frame>base_footprint</robot_base_frame>
-      <!-- Topics -->
-      <ros>
-        <remapping>cmd_vel:=/cmd_vel</remapping>
-        <remapping>odom:=/odom</remapping>
-      </ros>
-    </plugin>
-    <!-- Joint state publisher — required for robot_state_publisher -->
-    <plugin name="gazebo_ros_joint_state_publisher"
-            filename="libgazebo_ros_joint_state_publisher.so">
-      <update_rate>30</update_rate>
-      <joint_name>left_wheel_joint</joint_name>
-      <joint_name>right_wheel_joint</joint_name>
-    </plugin>
-  </gazebo>
-</robot>
+/home/betheln/ros2_ws/src/Robotics/delivery_robot2/build/delivery_robot/urdf/robot.urdf.xacro
